File: SplitSync/SplitSync.kicad_pcb (KiCad board)
At the start: 2 copper layers, 0 parts

Commit message: schematic for keyboard switches layout done.
Parts:
- added D1: Diode, ScottoKeebs_Components:Diode_SOD-123, B.Cu at (149.3, 33.2)
- added D10: Diode, ScottoKeebs_Components:Diode_SOD-123, B.Cu at (143.5, 36.5)
- added D11: Diode, ScottoKeebs_Components:Diode_SOD-123, B.Cu at (143.5, 39.9)
- added D12: Diode, ScottoKeebs_Components:Diode_SOD-123, B.Cu at (143.5, 43.2)
- added D13: Diode, ScottoKeebs_Components:Diode_SOD-123, B.Cu at (143.5, 46.6)
- added D14: Diode, ScottoKeebs_Components:Diode_SOD-123, B.Cu at (143.5, 49.9)
- added D15: Diode, ScottoKeebs_Components:Diode_SOD-123, B.Cu at (143.5, 53.3)
- added D16: Diode, ScottoKeebs_Components:Diode_SOD-123, B.Cu at (143.5, 56.6)
- added D17: Diode, ScottoKeebs_Components:Diode_SOD-123, B.Cu at (137.8, 33.2)
- added D18: Diode, ScottoKeebs_Components:Diode_SOD-123, B.Cu at (137.8, 36.5)
- added D19: Diode, ScottoKeebs_Components:Diode_SOD-123, B.Cu at (137.8, 39.9)
- added D2: Diode, ScottoKeebs_Components:Diode_SOD-123, B.Cu at (149.3, 36.5)
- added D20: Diode, ScottoKeebs_Components:Diode_SOD-123, B.Cu at (137.8, 43.2)
- added D21: Diode, ScottoKeebs_Components:Diode_SOD-123, B.Cu at (137.8, 46.6)
- added D22: Diode, ScottoKeebs_Components:Diode_SOD-123, B.Cu at (137.8, 49.9)
- added D23: Diode, ScottoKeebs_Components:Diode_SOD-123, B.Cu at (137.8, 53.3)
- added D24: Diode, ScottoKeebs_Components:Diode_SOD-123, B.Cu at (137.8, 56.6)
- added D25: Diode, ScottoKeebs_Components:Diode_SOD-123, B.Cu at (132.0, 33.2)
- added D26: Diode, ScottoKeebs_Components:Diode_SOD-123, B.Cu at (132.0, 36.5)
- added D27: Diode, ScottoKeebs_Components:Diode_SOD-123, B.Cu at (132.0, 39.9)
- added D28: Diode, ScottoKeebs_Components:Diode_SOD-123, B.Cu at (132.0, 43.2)
- added D29: Diode, ScottoKeebs_Components:Diode_SOD-123, B.Cu at (132.0, 46.6)
- added D3: Diode, ScottoKeebs_Components:Diode_SOD-123, B.Cu at (149.3, 39.9)
- added D30: Diode, ScottoKeebs_Components:Diode_SOD-123, B.Cu at (132.0, 49.9)
- added D31: Diode, ScottoKeebs_Components:Diode_SOD-123, B.Cu at (132.0, 53.3)
- added D32: Diode, ScottoKeebs_Components:Diode_SOD-123, B.Cu at (132.0, 56.6)
- added D33: Diode, ScottoKeebs_Components:Diode_SOD-123, B.Cu at (126.3, 33.2)
- added D34: Diode, ScottoKeebs_Components:Diode_SOD-123, B.Cu at (126.3, 36.5)
- added D35: Diode, ScottoKeebs_Components:Diode_SOD-123, B.Cu at (126.3, 39.9)
- added D36: Diode, ScottoKeebs_Components:Diode_SOD-123, B.Cu at (126.3, 43.2)
- added D37: Diode, ScottoKeebs_Components:Diode_SOD-123, B.Cu at (126.3, 46.6)
- added D38: Diode, ScottoKeebs_Components:Diode_SOD-123, B.Cu at (126.3, 49.9)
- added D39: Diode, ScottoKeebs_Components:Diode_SOD-123, B.Cu at (126.3, 53.3)
- added D4: Diode, ScottoKeebs_Components:Diode_SOD-123, B.Cu at (149.3, 43.2)
- added D40: Diode, ScottoKeebs_Components:Diode_SOD-123, B.Cu at (126.3, 56.6)
- added D5: Diode, ScottoKeebs_Components:Diode_SOD-123, B.Cu at (149.3, 46.6)
- added D6: Diode, ScottoKeebs_Components:Diode_SOD-123, B.Cu at (149.3, 49.9)
- added D7: Diode, ScottoKeebs_Components:Diode_SOD-123, B.Cu at (149.3, 53.3)
- added D8: Diode, ScottoKeebs_Components:Diode_SOD-123, B.Cu at (149.3, 56.6)
- added D9: Diode, ScottoKeebs_Components:Diode_SOD-123, B.Cu at (143.5, 33.2)
- added K_1: KEYSW, ScottoKeebs_Hotswap:Hotswap_MX_Plated_1.00u, F.Cu at (49.1, 39.3)
- added K_10: KEYSW, ScottoKeebs_Hotswap:Hotswap_MX_Plated_1.00u, F.Cu at (65.7, 54.8)
- added K_11: KEYSW, ScottoKeebs_Hotswap:Hotswap_MX_Plated_1.00u, F.Cu at (65.7, 70.4)
- added K_12: KEYSW, ScottoKeebs_Hotswap:Hotswap_MX_Plated_1.00u, F.Cu at (65.7, 85.9)
- added K_13: KEYSW, ScottoKeebs_Hotswap:Hotswap_MX_Plated_1.00u, F.Cu at (65.7, 101.5)
- added K_14: KEYSW, ScottoKeebs_Hotswap:Hotswap_MX_Plated_1.00u, F.Cu at (65.7, 117.0)
- added K_15: KEYSW, ScottoKeebs_Hotswap:Hotswap_MX_Plated_1.00u, F.Cu at (65.7, 132.6)
- added K_16: KEYSW, ScottoKeebs_Hotswap:Hotswap_MX_Plated_1.00u, F.Cu at (65.7, 148.1)
- added K_17: KEYSW, ScottoKeebs_Hotswap:Hotswap_MX_Plated_1.00u, F.Cu at (82.4, 39.3)
- added K_18: KEYSW, ScottoKeebs_Hotswap:Hotswap_MX_Plated_1.00u, F.Cu at (82.4, 54.8)
- added K_19: KEYSW, ScottoKeebs_Hotswap:Hotswap_MX_Plated_1.00u, F.Cu at (82.4, 70.4)
- added K_2: KEYSW, ScottoKeebs_Hotswap:Hotswap_MX_Plated_1.00u, F.Cu at (49.1, 54.8)
- added K_20: KEYSW, ScottoKeebs_Hotswap:Hotswap_MX_Plated_1.00u, F.Cu at (82.4, 85.9)
- added K_21: KEYSW, ScottoKeebs_Hotswap:Hotswap_MX_Plated_1.00u, F.Cu at (82.4, 101.5)
- added K_22: KEYSW, ScottoKeebs_Hotswap:Hotswap_MX_Plated_1.00u, F.Cu at (82.4, 117.0)
- added K_23: KEYSW, ScottoKeebs_Hotswap:Hotswap_MX_Plated_1.00u, F.Cu at (82.4, 132.6)
- added K_24: KEYSW, ScottoKeebs_Hotswap:Hotswap_MX_Plated_1.00u, F.Cu at (82.4, 148.1)
- added K_25: KEYSW, ScottoKeebs_Hotswap:Hotswap_MX_Plated_1.75u, F.Cu at (99.0, 39.3)
- added K_26: KEYSW, ScottoKeebs_Hotswap:Hotswap_MX_Plated_1.00u, F.Cu at (99.0, 54.8)
- added K_27: KEYSW, ScottoKeebs_Hotswap:Hotswap_MX_Plated_1.00u, F.Cu at (99.0, 70.4)
- added K_28: KEYSW, ScottoKeebs_Hotswap:Hotswap_MX_Plated_1.00u, F.Cu at (99.0, 85.9)
- added K_29: KEYSW, ScottoKeebs_Hotswap:Hotswap_MX_Plated_1.00u, F.Cu at (99.0, 101.5)
- added K_3: KEYSW, ScottoKeebs_Hotswap:Hotswap_MX_Plated_1.00u, F.Cu at (49.1, 70.4)
- added K_30: KEYSW, ScottoKeebs_Hotswap:Hotswap_MX_Plated_1.00u, F.Cu at (99.0, 117.0)
- added K_31: KEYSW, ScottoKeebs_Hotswap:Hotswap_MX_Plated_1.00u, F.Cu at (99.0, 132.6)
- added K_32: KEYSW, ScottoKeebs_Hotswap:Hotswap_MX_Plated_1.00u, F.Cu at (99.0, 148.1)
- added K_33: KEYSW, ScottoKeebs_Hotswap:Hotswap_MX_Plated_3.00u, F.Cu at (115.6, 39.3)
- added K_34: KEYSW, ScottoKeebs_Hotswap:Hotswap_MX_Plated_1.00u, F.Cu at (115.6, 54.8)
- added K_35: KEYSW, ScottoKeebs_Hotswap:Hotswap_MX_Plated_1.00u, F.Cu at (115.6, 70.4)
- added K_36: KEYSW, ScottoKeebs_Hotswap:Hotswap_MX_Plated_1.25u, F.Cu at (115.6, 85.9)
- added K_37: KEYSW, ScottoKeebs_Hotswap:Hotswap_MX_Plated_2.25u, F.Cu at (115.6, 101.5)
- added K_38: KEYSW, ScottoKeebs_Hotswap:Hotswap_MX_Plated_1.00u, F.Cu at (115.6, 117.0)
- added K_39: KEYSW, ScottoKeebs_Hotswap:Hotswap_MX_Plated_1.25u, F.Cu at (115.6, 132.6)
- added K_4: KEYSW, ScottoKeebs_Hotswap:Hotswap_MX_Plated_1.50u, F.Cu at (49.1, 85.9)
- added K_40: KEYSW, ScottoKeebs_Hotswap:Hotswap_MX_Plated_1.25u, F.Cu at (115.6, 148.1)
- added K_5: KEYSW, ScottoKeebs_Hotswap:Hotswap_MX_Plated_1.00u, F.Cu at (49.1, 101.5)
- added K_6: KEYSW, ScottoKeebs_Hotswap:Hotswap_MX_Plated_1.00u, F.Cu at (49.1, 117.0)
- added K_7: KEYSW, ScottoKeebs_Hotswap:Hotswap_MX_Plated_1.00u, F.Cu at (49.1, 132.6)
- added K_8: KEYSW, ScottoKeebs_Hotswap:Hotswap_MX_Plated_1.00u, F.Cu at (49.1, 148.1)
- added K_9: KEYSW, ScottoKeebs_Hotswap:Hotswap_MX_Plated_1.00u, F.Cu at (65.7, 39.3)

Commit message: layout setup entered and footprints assigned
Parts:
- removed D1, D10, D11, D12, D13, D14, D15, D16, D17, D18, D19, D2, D20, D21, D22, D23, D24, D25, D26, D27, D28, D29, D3, D30, D31, D32, D33, D34, D35, D36, D37, D38, D39, D4, D40, D5, D6, D7, D8, D9: Diode, ScottoKeebs_Components:Diode_SOD-123
- removed the K_1 at (49.1, 39.3)
- removed the K_10 at (65.7, 54.8)
- removed the K_11 at (65.7, 70.4)
- removed the K_12 at (65.7, 85.9)
- removed the K_13 at (65.7, 101.5)
- removed the K_14 at (65.7, 117.0)
- removed the K_15 at (65.7, 132.6)
- removed the K_16 at (65.7, 148.1)
- removed the K_17 at (82.4, 39.3)
- removed the K_18 at (82.4, 54.8)
- removed the K_19 at (82.4, 70.4)
- removed the K_2 at (49.1, 54.8)
- removed the K_20 at (82.4, 85.9)
- removed the K_21 at (82.4, 101.5)
- removed the K_22 at (82.4, 117.0)
- removed the K_23 at (82.4, 132.6)
- removed the K_24 at (82.4, 148.1)
- removed the K_25 at (99.0, 39.3)
- removed the K_26 at (99.0, 54.8)
- removed the K_27 at (99.0, 70.4)
- removed the K_28 at (99.0, 85.9)
- removed the K_29 at (99.0, 101.5)
- removed the K_3 at (49.1, 70.4)
- removed the K_30 at (99.0, 117.0)
- removed the K_31 at (99.0, 132.6)
- removed the K_32 at (99.0, 148.1)
- removed the K_33 at (115.6, 39.3)
- removed the K_34 at (115.6, 54.8)
- removed the K_35 at (115.6, 70.4)
- removed the K_36 at (115.6, 85.9)
- removed the K_37 at (115.6, 101.5)
- removed the K_38 at (115.6, 117.0)
- removed the K_39 at (115.6, 132.6)
- removed the K_4 at (49.1, 85.9)
- removed the K_5 at (49.1, 101.5)
- removed the K_6 at (49.1, 117.0)
- removed the K_7 at (49.1, 132.6)
- removed the K_8 at (49.1, 148.1)
- removed the K_9 at (65.7, 39.3)
- added D_0: D, Diode_SMD:D_SOD-123, B.Cu at (110.7, 155.6)
- added D_0: D, Diode_SMD:D_SOD-123, B.Cu at (317.1, 155.6)
- added D_1: D, Diode_SMD:D_SOD-123, B.Cu at (129.7, 155.6)
- added D_1: D, Diode_SMD:D_SOD-123, B.Cu at (336.2, 155.6)
- added D_10: D, Diode_SMD:D_SOD-123, B.Cu at (345.7, 174.6)
- added D_10: D, Diode_SMD:D_SOD-123, B.Cu at (125.0, 174.6)
- added D_11: D, Diode_SMD:D_SOD-123, B.Cu at (167.8, 174.6)
- added D_11: D, Diode_SMD:D_SOD-123, B.Cu at (364.7, 174.6)
- added D_12: D, Diode_SMD:D_SOD-123, B.Cu at (186.9, 174.6)
- added D_12: D, Diode_SMD:D_SOD-123, B.Cu at (383.8, 174.6)
- added D_13: D, Diode_SMD:D_SOD-123, B.Cu at (402.8, 174.6)
- added D_13: D, Diode_SMD:D_SOD-123, B.Cu at (205.9, 174.6)
- added D_14: D, Diode_SMD:D_SOD-123, B.Cu at (225.0, 174.6)
- added D_14: D, Diode_SMD:D_SOD-123, B.Cu at (421.9, 174.6)
- added D_15: D, Diode_SMD:D_SOD-123, B.Cu at (244.0, 174.6)
- added D_15: D, Diode_SMD:D_SOD-123, B.Cu at (450.5, 174.6)
- added D_16: D, Diode_SMD:D_SOD-123, B.Cu at (263.1, 174.6)
- added D_16: D, Diode_SMD:D_SOD-123, B.Cu at (483.8, 174.6)
- added D_17: D, Diode_SMD:D_SOD-123, B.Cu at (502.9, 174.6)
- added D_17: D, Diode_SMD:D_SOD-123, B.Cu at (282.1, 174.6)
- added D_18: D, Diode_SMD:D_SOD-123, B.Cu at (101.1, 193.7)
- added D_18: D, Diode_SMD:D_SOD-123, B.Cu at (312.4, 193.7)
- added D_19: D, Diode_SMD:D_SOD-123, B.Cu at (331.4, 193.7)
- added D_19: D, Diode_SMD:D_SOD-123, B.Cu at (120.2, 193.7)
- added D_2: D, Diode_SMD:D_SOD-123, B.Cu at (158.3, 155.6)
- added D_2: D, Diode_SMD:D_SOD-123, B.Cu at (355.2, 155.6)
- added D_20: D, Diode_SMD:D_SOD-123, B.Cu at (350.5, 193.7)
- added D_20: D, Diode_SMD:D_SOD-123, B.Cu at (172.6, 193.7)
- added D_21: D, Diode_SMD:D_SOD-123, B.Cu at (191.6, 193.7)
- added D_21: D, Diode_SMD:D_SOD-123, B.Cu at (369.5, 193.7)
- added D_22: D, Diode_SMD:D_SOD-123, B.Cu at (388.6, 193.7)
- added D_22: D, Diode_SMD:D_SOD-123, B.Cu at (210.7, 193.7)
- added D_23: D, Diode_SMD:D_SOD-123, B.Cu at (407.6, 193.7)
- added D_23: D, Diode_SMD:D_SOD-123, B.Cu at (229.7, 193.7)
- added D_24: D, Diode_SMD:D_SOD-123, B.Cu at (248.8, 193.7)
- added D_24: D, Diode_SMD:D_SOD-123, B.Cu at (450.5, 193.7)
- added D_25: D, Diode_SMD:D_SOD-123, B.Cu at (488.6, 193.7)
- added D_25: D, Diode_SMD:D_SOD-123, B.Cu at (267.8, 193.7)
- added D_26: D, Diode_SMD:D_SOD-123, B.Cu at (507.6, 193.7)
- added D_26: D, Diode_SMD:D_SOD-123, B.Cu at (105.9, 212.7)
- added D_27: D, Diode_SMD:D_SOD-123, B.Cu at (125.0, 212.7)
- added D_27: D, Diode_SMD:D_SOD-123, B.Cu at (321.9, 212.7)
- added D_28: D, Diode_SMD:D_SOD-123, B.Cu at (182.1, 212.7)
- added D_28: D, Diode_SMD:D_SOD-123, B.Cu at (340.9, 212.7)
- added D_29: D, Diode_SMD:D_SOD-123, B.Cu at (201.2, 212.7)
- added D_29: D, Diode_SMD:D_SOD-123, B.Cu at (360.0, 212.7)
- added D_3: D, Diode_SMD:D_SOD-123, B.Cu at (177.3, 155.6)
- added D_3: D, Diode_SMD:D_SOD-123, B.Cu at (374.3, 155.6)
- added D_30: D, Diode_SMD:D_SOD-123, B.Cu at (379.0, 212.7)
- added D_30: D, Diode_SMD:D_SOD-123, B.Cu at (220.2, 212.7)
- added D_31: D, Diode_SMD:D_SOD-123, B.Cu at (398.1, 212.7)
- added D_31: D, Diode_SMD:D_SOD-123, B.Cu at (239.3, 212.7)
- added D_32: D, Diode_SMD:D_SOD-123, B.Cu at (450.5, 212.7)
- added D_32: D, Diode_SMD:D_SOD-123, B.Cu at (258.3, 212.7)
- added D_33: D, Diode_SMD:D_SOD-123, B.Cu at (483.8, 212.7)
- added D_33: D, Diode_SMD:D_SOD-123, B.Cu at (277.4, 212.7)
- added D_34: D, Diode_SMD:D_SOD-123, B.Cu at (502.9, 212.7)
- added D_34: D, Diode_SMD:D_SOD-123, B.Cu at (110.7, 231.8)
- added D_35: D, Diode_SMD:D_SOD-123, B.Cu at (129.7, 231.8)
- added D_35: D, Diode_SMD:D_SOD-123, B.Cu at (350.5, 231.8)
- added D_36: D, Diode_SMD:D_SOD-123, B.Cu at (374.3, 231.8)
- added D_36: D, Diode_SMD:D_SOD-123, B.Cu at (163.1, 231.8)
- added D_37: D, Diode_SMD:D_SOD-123, B.Cu at (398.1, 231.8)
- added D_37: D, Diode_SMD:D_SOD-123, B.Cu at (186.9, 231.8)
- added D_38: D, Diode_SMD:D_SOD-123, B.Cu at (421.9, 231.8)
- added D_38: D, Diode_SMD:D_SOD-123, B.Cu at (210.7, 231.8)
- added D_39: D, Diode_SMD:D_SOD-123, B.Cu at (267.8, 231.8)
- added D_39: D, Diode_SMD:D_SOD-123, B.Cu at (450.5, 231.8)
- added D_4: D, Diode_SMD:D_SOD-123, B.Cu at (196.4, 155.6)
- added D_4: D, Diode_SMD:D_SOD-123, B.Cu at (393.3, 155.6)
- added D_40: D, Diode_SMD:D_SOD-123, B.Cu at (479.0, 231.8)
- added D_41: D, Diode_SMD:D_SOD-123, B.Cu at (498.1, 231.8)
- added D_5: D, Diode_SMD:D_SOD-123, B.Cu at (412.4, 155.6)
- added D_5: D, Diode_SMD:D_SOD-123, B.Cu at (215.4, 155.6)
- added D_6: D, Diode_SMD:D_SOD-123, B.Cu at (234.5, 155.6)
- added D_6: D, Diode_SMD:D_SOD-123, B.Cu at (450.5, 155.6)
- added D_7: D, Diode_SMD:D_SOD-123, B.Cu at (479.0, 155.6)
- added D_7: D, Diode_SMD:D_SOD-123, B.Cu at (253.5, 155.6)
- added D_8: D, Diode_SMD:D_SOD-123, B.Cu at (498.1, 155.6)
- added D_8: D, Diode_SMD:D_SOD-123, B.Cu at (272.6, 155.6)
- added D_9: D, Diode_SMD:D_SOD-123, B.Cu at (105.9, 174.6)
- added D_9: D, Diode_SMD:D_SOD-123, B.Cu at (326.6, 174.6)
- added K_0: KEYSW, MX_Alps_Hybrid:MX-1U-NoLED, F.Cu at (308.6, 155.1)
- added K_0: KEYSW, MX_Alps_Hybrid:MX-1U-NoLED, F.Cu at (102.1, 155.1)
- added K_1: KEYSW, MX_Alps_Hybrid:MX-1U-NoLED, F.Cu at (121.2, 155.1)
- added K_1: KEYSW, MX_Alps_Hybrid:MX-1U-NoLED, F.Cu at (327.6, 155.1)
- added K_10: KEYSW, MX_Alps_Hybrid:MX-1U-NoLED, F.Cu at (116.4, 174.1)
- added K_10: KEYSW, MX_Alps_Hybrid:MX-1U-NoLED, F.Cu at (337.2, 174.1)
- added K_11: KEYSW, MX_Alps_Hybrid:MX-1U-NoLED, F.Cu at (356.2, 174.1)
- added K_11: KEYSW, MX_Alps_Hybrid:MX-1.5U-NoLED, F.Cu at (154.5, 174.1)
- added K_12: KEYSW, MX_Alps_Hybrid:MX-1U-NoLED, F.Cu at (375.3, 174.1)
- added K_12: KEYSW, MX_Alps_Hybrid:MX-1U-NoLED, F.Cu at (178.3, 174.1)
- added K_13: KEYSW, MX_Alps_Hybrid:MX-1U-NoLED, F.Cu at (197.4, 174.1)
- added K_13: KEYSW, MX_Alps_Hybrid:MX-1U-NoLED, F.Cu at (394.3, 174.1)
- added K_14: KEYSW, MX_Alps_Hybrid:MX-1U-NoLED, F.Cu at (413.4, 174.1)
- added K_14: KEYSW, MX_Alps_Hybrid:MX-1U-NoLED, F.Cu at (216.4, 174.1)
- added K_15: KEYSW, MX_Alps_Hybrid:MX-1U-NoLED, F.Cu at (235.5, 174.1)
- added K_15: KEYSW, MX_Alps_Hybrid:MX-1.5U-NoLED, F.Cu at (437.2, 174.1)
- added K_16: KEYSW, MX_Alps_Hybrid:MX-1U-NoLED, F.Cu at (254.5, 174.1)
- added K_16: KEYSW, MX_Alps_Hybrid:MX-1U-NoLED, F.Cu at (475.3, 174.1)
- added K_17: KEYSW, MX_Alps_Hybrid:MX-1U-NoLED, F.Cu at (273.6, 174.1)
- added K_17: KEYSW, MX_Alps_Hybrid:MX-1U-NoLED, F.Cu at (494.3, 174.1)
- added K_18: KEYSW, MX_Alps_Hybrid:MX-1U-NoLED, F.Cu at (303.8, 193.2)
- added K_18: KEYSW, MX_Alps_Hybrid:MX-1U-NoLED, F.Cu at (92.6, 193.2)
- added K_19: KEYSW, MX_Alps_Hybrid:MX-1U-NoLED, F.Cu at (111.7, 193.2)
- added K_19: KEYSW, MX_Alps_Hybrid:MX-1U-NoLED, F.Cu at (322.9, 193.2)
- added K_2: KEYSW, MX_Alps_Hybrid:MX-1U-NoLED, F.Cu at (346.7, 155.1)
- added K_2: KEYSW, MX_Alps_Hybrid:MX-1U-NoLED, F.Cu at (149.8, 155.1)
- added K_20: KEYSW, MX_Alps_Hybrid:MX-1.75U-NoLED, F.Cu at (156.9, 193.2)
- added K_20: KEYSW, MX_Alps_Hybrid:MX-1U-NoLED, F.Cu at (341.9, 193.2)
- added K_21: KEYSW, MX_Alps_Hybrid:MX-1U-NoLED, F.Cu at (183.1, 193.2)
- added K_21: KEYSW, MX_Alps_Hybrid:MX-1U-NoLED, F.Cu at (361.0, 193.2)
- added K_22: KEYSW, MX_Alps_Hybrid:MX-1U-NoLED, F.Cu at (202.2, 193.2)
- added K_22: KEYSW, MX_Alps_Hybrid:MX-1U-NoLED, F.Cu at (380.0, 193.2)
- added K_23: KEYSW, MX_Alps_Hybrid:MX-1U-NoLED, F.Cu at (221.2, 193.2)
- added K_23: KEYSW, MX_Alps_Hybrid:MX-1U-NoLED, F.Cu at (399.1, 193.2)
- added K_24: KEYSW, MX_Alps_Hybrid:MX-2.25U-NoLED, F.Cu at (430.0, 193.2)
- added K_24: KEYSW, MX_Alps_Hybrid:MX-1U-NoLED, F.Cu at (240.3, 193.2)
- added K_25: KEYSW, MX_Alps_Hybrid:MX-1U-NoLED, F.Cu at (480.0, 193.2)
- added K_25: KEYSW, MX_Alps_Hybrid:MX-1U-NoLED, F.Cu at (259.3, 193.2)
- added K_26: KEYSW, MX_Alps_Hybrid:MX-1U-NoLED, F.Cu at (97.4, 212.2)
- added K_26: KEYSW, MX_Alps_Hybrid:MX-1U-NoLED, F.Cu at (499.1, 193.2)
- added K_27: KEYSW, MX_Alps_Hybrid:MX-1U-NoLED, F.Cu at (116.4, 212.2)
- added K_27: KEYSW, MX_Alps_Hybrid:MX-1U-NoLED, F.Cu at (313.4, 212.2)
- added K_28: KEYSW, MX_Alps_Hybrid:MX-1U-NoLED, F.Cu at (332.4, 212.2)
- added K_28: KEYSW, MX_Alps_Hybrid:MX-2.25U-NoLED, F.Cu at (161.7, 212.2)
- added K_29: KEYSW, MX_Alps_Hybrid:MX-1U-NoLED, F.Cu at (192.6, 212.2)
- added K_29: KEYSW, MX_Alps_Hybrid:MX-1U-NoLED, F.Cu at (351.5, 212.2)
- added K_3: KEYSW, MX_Alps_Hybrid:MX-1U-NoLED, F.Cu at (365.7, 155.1)
- added K_3: KEYSW, MX_Alps_Hybrid:MX-1U-NoLED, F.Cu at (168.8, 155.1)
- added K_30: KEYSW, MX_Alps_Hybrid:MX-1U-NoLED, F.Cu at (370.5, 212.2)
- added K_30: KEYSW, MX_Alps_Hybrid:MX-1U-NoLED, F.Cu at (211.7, 212.2)
- added K_31: KEYSW, MX_Alps_Hybrid:MX-1U-NoLED, F.Cu at (230.7, 212.2)
- added K_31: KEYSW, MX_Alps_Hybrid:MX-1U-NoLED, F.Cu at (389.6, 212.2)
- added K_32: KEYSW, MX_Alps_Hybrid:MX-1U-NoLED, F.Cu at (249.8, 212.2)
- added K_32: KEYSW, MX_Alps_Hybrid:MX-2.75U-NoLED, F.Cu at (425.3, 212.2)
- added K_33: KEYSW, MX_Alps_Hybrid:MX-1U-NoLED, F.Cu at (268.8, 212.2)
- added K_33: KEYSW, MX_Alps_Hybrid:MX-1U-NoLED, F.Cu at (475.3, 212.2)
- added K_34: KEYSW, MX_Alps_Hybrid:MX-1U-NoLED, F.Cu at (494.3, 212.2)
- added K_34: KEYSW, MX_Alps_Hybrid:MX-1U-NoLED, F.Cu at (102.1, 231.3)
- added K_35: KEYSW, MX_Alps_Hybrid:MX-1U-NoLED, F.Cu at (121.2, 231.3)
- added K_35: KEYSW, MX_Alps_Hybrid:MX-3U-NoLED, F.Cu at (322.9, 231.3)
- added K_36: KEYSW, MX_Alps_Hybrid:MX-1.25U-NoLED, F.Cu at (363.4, 231.3)
- added K_36: KEYSW, MX_Alps_Hybrid:MX-1.25U-NoLED, F.Cu at (152.2, 231.3)
- added K_37: KEYSW, MX_Alps_Hybrid:MX-1.25U-NoLED, F.Cu at (387.2, 231.3)
- added K_37: KEYSW, MX_Alps_Hybrid:MX-1.25U-NoLED, F.Cu at (176.0, 231.3)
- added K_38: KEYSW, MX_Alps_Hybrid:MX-1.25U-NoLED, F.Cu at (199.8, 231.3)
- added K_38: KEYSW, MX_Alps_Hybrid:MX-1.25U-NoLED, F.Cu at (411.0, 231.3)
- added K_39: KEYSW, MX_Alps_Hybrid:MX-1.5U-NoLED, F.Cu at (437.2, 231.3)
- added K_39: KEYSW, MX_Alps_Hybrid:MX-3U-NoLED, F.Cu at (240.3, 231.3)
- added K_4: KEYSW, MX_Alps_Hybrid:MX-1U-NoLED, F.Cu at (187.9, 155.1)
- added K_4: KEYSW, MX_Alps_Hybrid:MX-1U-NoLED, F.Cu at (384.8, 155.1)
- added K_41: KEYSW, MX_Alps_Hybrid:MX-1U-NoLED, F.Cu at (489.6, 231.3)
- added K_5: KEYSW, MX_Alps_Hybrid:MX-1U-NoLED, F.Cu at (206.9, 155.1)
- added K_5: KEYSW, MX_Alps_Hybrid:MX-1U-NoLED, F.Cu at (403.8, 155.1)
- added K_6: KEYSW, MX_Alps_Hybrid:MX-1U-NoLED, F.Cu at (226.0, 155.1)
- added K_6: KEYSW, MX_Alps_Hybrid:MX-2U-NoLED, F.Cu at (432.4, 155.1)
- added K_7: KEYSW, MX_Alps_Hybrid:MX-1U-NoLED, F.Cu at (245.0, 155.1)
- added K_7: KEYSW, MX_Alps_Hybrid:MX-1U-NoLED, F.Cu at (470.5, 155.1)
- added K_8: KEYSW, MX_Alps_Hybrid:MX-1U-NoLED, F.Cu at (489.6, 155.1)
- added K_8: KEYSW, MX_Alps_Hybrid:MX-1U-NoLED, F.Cu at (264.1, 155.1)
- added K_9: KEYSW, MX_Alps_Hybrid:MX-1U-NoLED, F.Cu at (318.1, 174.1)
- added K_9: KEYSW, MX_Alps_Hybrid:MX-1U-NoLED, F.Cu at (97.4, 174.1)
- K_40: footprint ScottoKeebs_Hotswap:Hotswap_MX_Plated_1.25u -> MX_Alps_Hybrid:MX-1U-NoLED
- moved K_40 364.5 mm to (470.5, 231.3)
Connections:
- K_40 pad 1: col8 -> col5

Commit message: components laid out.
Parts:
- removed the D_0 at (110.7, 155.6)
- removed the D_0 at (317.1, 155.6)
- removed the D_1 at (129.7, 155.6)
- removed the D_1 at (336.2, 155.6)
- removed the D_10 at (345.7, 174.6)
- removed the D_10 at (125.0, 174.6)
- removed the D_11 at (167.8, 174.6)
- removed the D_11 at (364.7, 174.6)
- removed the D_12 at (186.9, 174.6)
- removed the D_12 at (383.8, 174.6)
- removed the D_13 at (402.8, 174.6)
- removed the D_13 at (205.9, 174.6)
- removed the D_14 at (225.0, 174.6)
- removed the D_14 at (421.9, 174.6)
- removed the D_15 at (244.0, 174.6)
- removed the D_15 at (450.5, 174.6)
- removed the D_16 at (263.1, 174.6)
- removed the D_16 at (483.8, 174.6)
- removed the D_17 at (502.9, 174.6)
- removed the D_17 at (282.1, 174.6)
- removed the D_18 at (101.1, 193.7)
- removed the D_18 at (312.4, 193.7)
- removed the D_19 at (331.4, 193.7)
- removed the D_19 at (120.2, 193.7)
- removed the D_2 at (158.3, 155.6)
- removed the D_2 at (355.2, 155.6)
- removed the D_20 at (350.5, 193.7)
- removed the D_20 at (172.6, 193.7)
- removed the D_21 at (191.6, 193.7)
- removed the D_21 at (369.5, 193.7)
- removed the D_22 at (388.6, 193.7)
- removed the D_22 at (210.7, 193.7)
- removed the D_23 at (407.6, 193.7)
- removed the D_23 at (229.7, 193.7)
- removed the D_24 at (248.8, 193.7)
- removed the D_24 at (450.5, 193.7)
- removed the D_25 at (488.6, 193.7)
- removed the D_25 at (267.8, 193.7)
- removed the D_26 at (507.6, 193.7)
- removed the D_26 at (105.9, 212.7)
- removed the D_27 at (125.0, 212.7)
- removed the D_27 at (321.9, 212.7)
- removed the D_28 at (182.1, 212.7)
- removed the D_28 at (340.9, 212.7)
- removed the D_29 at (201.2, 212.7)
- removed the D_29 at (360.0, 212.7)
- removed the D_3 at (177.3, 155.6)
- removed the D_3 at (374.3, 155.6)
- removed the D_30 at (379.0, 212.7)
- removed the D_30 at (220.2, 212.7)
- removed the D_31 at (398.1, 212.7)
- removed the D_31 at (239.3, 212.7)
- removed the D_32 at (450.5, 212.7)
- removed the D_32 at (258.3, 212.7)
- removed the D_33 at (483.8, 212.7)
- removed the D_33 at (277.4, 212.7)
- removed the D_34 at (502.9, 212.7)
- removed the D_34 at (110.7, 231.8)
- removed the D_35 at (129.7, 231.8)
- removed the D_35 at (350.5, 231.8)
- removed the D_36 at (374.3, 231.8)
- removed the D_36 at (163.1, 231.8)
- removed the D_37 at (398.1, 231.8)
- removed the D_37 at (186.9, 231.8)
- removed the D_38 at (421.9, 231.8)
- removed the D_38 at (210.7, 231.8)
- removed the D_39 at (267.8, 231.8)
- removed the D_39 at (450.5, 231.8)
- removed the D_4 at (196.4, 155.6)
- removed the D_4 at (393.3, 155.6)
- removed the D_5 at (412.4, 155.6)
- removed the D_5 at (215.4, 155.6)
- removed the D_6 at (234.5, 155.6)
- removed the D_6 at (450.5, 155.6)
- removed the D_7 at (479.0, 155.6)
- removed the D_7 at (253.5, 155.6)
- removed the D_8 at (498.1, 155.6)
- removed the D_8 at (272.6, 155.6)
- removed the D_9 at (105.9, 174.6)
- removed the D_9 at (326.6, 174.6)
- removed the K_0 at (308.6, 155.1)
- removed the K_0 at (102.1, 155.1)
- removed the K_1 at (121.2, 155.1)
- removed the K_1 at (327.6, 155.1)
- removed the K_10 at (116.4, 174.1)
- removed the K_10 at (337.2, 174.1)
- removed the K_11 at (356.2, 174.1)
- removed the K_11 at (154.5, 174.1)
- removed the K_12 at (375.3, 174.1)
- removed the K_12 at (178.3, 174.1)
- removed the K_13 at (197.4, 174.1)
- removed the K_13 at (394.3, 174.1)
- removed the K_14 at (413.4, 174.1)
- removed the K_14 at (216.4, 174.1)
- removed the K_15 at (235.5, 174.1)
- removed the K_15 at (437.2, 174.1)
- removed the K_16 at (254.5, 174.1)
- removed the K_16 at (475.3, 174.1)
- removed the K_17 at (273.6, 174.1)
- removed the K_17 at (494.3, 174.1)
- removed the K_18 at (303.8, 193.2)
- removed the K_18 at (92.6, 193.2)
- removed the K_19 at (111.7, 193.2)
- removed the K_19 at (322.9, 193.2)
- removed the K_2 at (346.7, 155.1)
- removed the K_2 at (149.8, 155.1)
- removed the K_20 at (156.9, 193.2)
- removed the K_20 at (341.9, 193.2)
- removed the K_21 at (183.1, 193.2)
- removed the K_21 at (361.0, 193.2)
- removed the K_22 at (202.2, 193.2)
- removed the K_22 at (380.0, 193.2)
- removed the K_23 at (221.2, 193.2)
- removed the K_23 at (399.1, 193.2)
- removed the K_24 at (430.0, 193.2)
- removed the K_24 at (240.3, 193.2)
- removed the K_25 at (480.0, 193.2)
- removed the K_25 at (259.3, 193.2)
- removed the K_26 at (97.4, 212.2)
- removed the K_26 at (499.1, 193.2)
- removed the K_27 at (116.4, 212.2)
- removed the K_27 at (313.4, 212.2)
- removed the K_28 at (332.4, 212.2)
- removed the K_28 at (161.7, 212.2)
- removed the K_29 at (192.6, 212.2)
- removed the K_29 at (351.5, 212.2)
- removed the K_3 at (365.7, 155.1)
- removed the K_3 at (168.8, 155.1)
- removed the K_30 at (370.5, 212.2)
- removed the K_30 at (211.7, 212.2)
- removed the K_31 at (230.7, 212.2)
- removed the K_31 at (389.6, 212.2)
- removed the K_32 at (249.8, 212.2)
- removed the K_32 at (425.3, 212.2)
- removed the K_33 at (268.8, 212.2)
- removed the K_33 at (475.3, 212.2)
- removed the K_34 at (494.3, 212.2)
- removed the K_34 at (102.1, 231.3)
- removed the K_35 at (121.2, 231.3)
- removed the K_35 at (322.9, 231.3)
- removed the K_36 at (363.4, 231.3)
- removed the K_36 at (152.2, 231.3)
- removed the K_37 at (387.2, 231.3)
- removed the K_37 at (176.0, 231.3)
- removed the K_38 at (199.8, 231.3)
- removed the K_38 at (411.0, 231.3)
- removed the K_39 at (437.2, 231.3)
- removed the K_39 at (240.3, 231.3)
- removed the K_4 at (187.9, 155.1)
- removed the K_4 at (384.8, 155.1)
- removed the K_5 at (206.9, 155.1)
- removed the K_5 at (403.8, 155.1)
- removed the K_6 at (226.0, 155.1)
- removed the K_6 at (432.4, 155.1)
- removed the K_7 at (245.0, 155.1)
- removed the K_7 at (470.5, 155.1)
- removed the K_8 at (489.6, 155.1)
- removed the K_8 at (264.1, 155.1)
- removed the K_9 at (318.1, 174.1)
- removed the K_9 at (97.4, 174.1)
- added D_0: D, Diode_SMD:D_SOD-123, B.Cu at (110.4, 161.7)
- added D_1: D, Diode_SMD:D_SOD-123, B.Cu at (129.5, 161.7)
- added D_10: D, Diode_SMD:D_SOD-123, B.Cu at (335.0, 161.7)
- added D_11: D, Diode_SMD:D_SOD-123, B.Cu at (354.0, 161.7)
- added D_12: D, Diode_SMD:D_SOD-123, B.Cu at (373.1, 161.7)
- added D_13: D, Diode_SMD:D_SOD-123, B.Cu at (392.1, 161.7)
- added D_14: D, Diode_SMD:D_SOD-123, B.Cu at (411.2, 161.7)
- added D_15: D, Diode_SMD:D_SOD-123, B.Cu at (449.3, 161.7)
- added D_16: D, Diode_SMD:D_SOD-123, B.Cu at (478.1, 155.3)
- added D_17: D, Diode_SMD:D_SOD-123, B.Cu at (496.9, 155.3)
- added D_18: D, Diode_SMD:D_SOD-123, B.Cu at (105.7, 180.8)
- added D_19: D, Diode_SMD:D_SOD-123, B.Cu at (124.7, 180.8)
- added D_2: D, Diode_SMD:D_SOD-123, B.Cu at (158.0, 161.7)
- added D_20: D, Diode_SMD:D_SOD-123, B.Cu at (167.6, 180.8)
- added D_21: D, Diode_SMD:D_SOD-123, B.Cu at (186.6, 180.8)
- added D_22: D, Diode_SMD:D_SOD-123, B.Cu at (205.7, 180.8)
- added D_23: D, Diode_SMD:D_SOD-123, B.Cu at (224.7, 180.8)
- added D_24: D, Diode_SMD:D_SOD-123, B.Cu at (243.8, 180.8)
- added D_25: D, Diode_SMD:D_SOD-123, B.Cu at (262.8, 180.8)
- added D_26: D, Diode_SMD:D_SOD-123, B.Cu at (281.6, 180.7)
- added D_27: D, Diode_SMD:D_SOD-123, B.Cu at (325.4, 180.8)
- added D_28: D, Diode_SMD:D_SOD-123, B.Cu at (344.5, 180.8)
- added D_29: D, Diode_SMD:D_SOD-123, B.Cu at (363.5, 180.8)
- added D_3: D, Diode_SMD:D_SOD-123, B.Cu at (177.1, 161.7)
- added D_30: D, Diode_SMD:D_SOD-123, B.Cu at (382.6, 180.8)
- added D_31: D, Diode_SMD:D_SOD-123, B.Cu at (401.6, 180.8)
- added D_32: D, Diode_SMD:D_SOD-123, B.Cu at (420.7, 180.8)
- added D_33: D, Diode_SMD:D_SOD-123, B.Cu at (449.3, 180.8)
- added D_34: D, Diode_SMD:D_SOD-123, B.Cu at (482.6, 180.8)
- added D_35: D, Diode_SMD:D_SOD-123, B.Cu at (501.4, 180.8)
- added D_36: D, Diode_SMD:D_SOD-123, B.Cu at (100.9, 199.8)
- added D_37: D, Diode_SMD:D_SOD-123, B.Cu at (119.9, 199.8)
- added D_38: D, Diode_SMD:D_SOD-123, B.Cu at (172.3, 199.8)
- added D_39: D, Diode_SMD:D_SOD-123, B.Cu at (191.4, 199.8)
- added D_4: D, Diode_SMD:D_SOD-123, B.Cu at (196.1, 161.7)
- added D_42: D, Diode_SMD:D_SOD-123, B.Cu at (248.5, 199.8)
- added D_43: D, Diode_SMD:D_SOD-123, B.Cu at (267.3, 199.8)
- added D_44: D, Diode_SMD:D_SOD-123, B.Cu at (311.1, 199.8)
- added D_45: D, Diode_SMD:D_SOD-123, B.Cu at (330.2, 199.8)
- added D_46: D, Diode_SMD:D_SOD-123, B.Cu at (349.2, 199.8)
- added D_47: D, Diode_SMD:D_SOD-123, B.Cu at (368.3, 199.8)
- added D_48: D, Diode_SMD:D_SOD-123, B.Cu at (387.3, 199.8)
- added D_49: D, Diode_SMD:D_SOD-123, B.Cu at (406.4, 199.8)
- added D_5: D, Diode_SMD:D_SOD-123, B.Cu at (215.2, 161.7)
- added D_50: D, Diode_SMD:D_SOD-123, B.Cu at (449.3, 199.8)
- added D_51: D, Diode_SMD:D_SOD-123, B.Cu at (487.4, 199.8)
- added D_52: D, Diode_SMD:D_SOD-123, B.Cu at (506.1, 199.8)
- added D_53: D, Diode_SMD:D_SOD-123, B.Cu at (105.7, 218.9)
- added D_54: D, Diode_SMD:D_SOD-123, B.Cu at (124.7, 218.9)
- added D_55: D, Diode_SMD:D_SOD-123, B.Cu at (181.9, 218.9)
- added D_56: D, Diode_SMD:D_SOD-123, B.Cu at (200.9, 218.9)
- added D_57: D, Diode_SMD:D_SOD-123, B.Cu at (220.0, 218.9)
- added D_58: D, Diode_SMD:D_SOD-123, B.Cu at (239.0, 218.9)
- added D_59: D, Diode_SMD:D_SOD-123, B.Cu at (258.1, 218.9)
- added D_6: D, Diode_SMD:D_SOD-123, B.Cu at (234.2, 161.7)
- added D_60: D, Diode_SMD:D_SOD-123, B.Cu at (276.9, 218.8)
- added D_61: D, Diode_SMD:D_SOD-123, B.Cu at (320.7, 218.9)
- added D_62: D, Diode_SMD:D_SOD-123, B.Cu at (339.7, 218.9)
- added D_63: D, Diode_SMD:D_SOD-123, B.Cu at (358.8, 218.9)
- added D_64: D, Diode_SMD:D_SOD-123, B.Cu at (377.8, 218.9)
- added D_65: D, Diode_SMD:D_SOD-123, B.Cu at (396.9, 218.9)
- added D_66: D, Diode_SMD:D_SOD-123, B.Cu at (449.3, 218.9)
- added D_67: D, Diode_SMD:D_SOD-123, B.Cu at (482.6, 218.9)
- added D_68: D, Diode_SMD:D_SOD-123, B.Cu at (501.4, 218.9)
- added D_69: D, Diode_SMD:D_SOD-123, B.Cu at (110.4, 237.9)
- added D_7: D, Diode_SMD:D_SOD-123, B.Cu at (253.3, 161.7)
- added D_70: D, Diode_SMD:D_SOD-123, B.Cu at (129.5, 237.9)
- added D_71: D, Diode_SMD:D_SOD-123, B.Cu at (162.8, 237.9)
- added D_72: D, Diode_SMD:D_SOD-123, B.Cu at (186.6, 237.9)
- added D_73: D, Diode_SMD:D_SOD-123, B.Cu at (210.4, 237.9)
- added D_74: D, Diode_SMD:D_SOD-123, B.Cu at (267.3, 237.9)
- added D_75: D, Diode_SMD:D_SOD-123, B.Cu at (349.2, 237.9)
- added D_76: D, Diode_SMD:D_SOD-123, B.Cu at (373.1, 237.9)
- added D_77: D, Diode_SMD:D_SOD-123, B.Cu at (396.9, 237.9)
- added D_78: D, Diode_SMD:D_SOD-123, B.Cu at (420.7, 237.9)
- added D_79: D, Diode_SMD:D_SOD-123, B.Cu at (449.3, 237.9)
- added D_8: D, Diode_SMD:D_SOD-123, B.Cu at (272.1, 161.7)
- added D_80: D, Diode_SMD:D_SOD-123, B.Cu at (477.8, 237.9)
- added D_81: D, Diode_SMD:D_SOD-123, B.Cu at (496.6, 237.9)
- added D_9: D, Diode_SMD:D_SOD-123, B.Cu at (315.9, 161.7)
- added K_0: KEYSW, ScottoKeebs_Hotswap:Hotswap_MX_Plated_1.00u, F.Cu at (102.2, 154.8)
- added K_1: KEYSW, ScottoKeebs_Hotswap:Hotswap_MX_Plated_1.00u, F.Cu at (121.3, 154.8)
- added K_10: KEYSW, ScottoKeebs_Hotswap:Hotswap_MX_Plated_1.00u, F.Cu at (326.7, 154.8)
- added K_11: KEYSW, ScottoKeebs_Hotswap:Hotswap_MX_Plated_1.00u, F.Cu at (345.8, 154.8)
- added K_12: KEYSW, ScottoKeebs_Hotswap:Hotswap_MX_Plated_1.00u, F.Cu at (364.8, 154.8)
- added K_13: KEYSW, ScottoKeebs_Hotswap:Hotswap_MX_Plated_1.00u, F.Cu at (383.9, 154.8)
- added K_14: KEYSW, ScottoKeebs_Hotswap:Hotswap_MX_Plated_1.00u, F.Cu at (402.9, 154.8)
- added K_15: KEYSW, ScottoKeebs_Hotswap:Hotswap_MX_Plated_1.00u, F.Cu at (431.5, 154.8)
- added K_16: KEYSW, ScottoKeebs_Hotswap:Hotswap_MX_Plated_1.00u, F.Cu at (469.6, 154.8)
- added K_17: KEYSW, ScottoKeebs_Hotswap:Hotswap_MX_Plated_1.00u, F.Cu at (488.7, 154.8)
- added K_18: KEYSW, ScottoKeebs_Hotswap:Hotswap_MX_Plated_1.00u, F.Cu at (97.4, 173.9)
- added K_19: KEYSW, ScottoKeebs_Hotswap:Hotswap_MX_Plated_1.00u, F.Cu at (116.5, 173.9)
- added K_2: KEYSW, ScottoKeebs_Hotswap:Hotswap_MX_Plated_1.00u, F.Cu at (149.8, 154.8)
- added K_20: KEYSW, ScottoKeebs_Hotswap:Hotswap_MX_Plated_1.50u, F.Cu at (154.6, 173.9)
- added K_21: KEYSW, ScottoKeebs_Hotswap:Hotswap_MX_Plated_1.00u, F.Cu at (178.4, 173.9)
- added K_22: KEYSW, ScottoKeebs_Hotswap:Hotswap_MX_Plated_1.00u, F.Cu at (197.5, 173.9)
- added K_23: KEYSW, ScottoKeebs_Hotswap:Hotswap_MX_Plated_1.00u, F.Cu at (216.5, 173.9)
- added K_24: KEYSW, ScottoKeebs_Hotswap:Hotswap_MX_Plated_1.00u, F.Cu at (235.6, 173.9)
- added K_25: KEYSW, ScottoKeebs_Hotswap:Hotswap_MX_Plated_1.00u, F.Cu at (254.6, 173.9)
- added K_26: KEYSW, ScottoKeebs_Hotswap:Hotswap_MX_Plated_1.00u, F.Cu at (273.7, 173.9)
- added K_27: KEYSW, ScottoKeebs_Hotswap:Hotswap_MX_Plated_1.00u, F.Cu at (317.2, 173.9)
- added K_28: KEYSW, ScottoKeebs_Hotswap:Hotswap_MX_Plated_1.00u, F.Cu at (336.3, 173.9)
- added K_29: KEYSW, ScottoKeebs_Hotswap:Hotswap_MX_Plated_1.00u, F.Cu at (355.3, 173.9)
- added K_3: KEYSW, ScottoKeebs_Hotswap:Hotswap_MX_Plated_1.00u, F.Cu at (168.9, 154.8)
- added K_30: KEYSW, ScottoKeebs_Hotswap:Hotswap_MX_Plated_1.00u, F.Cu at (374.4, 173.9)
- added K_31: KEYSW, ScottoKeebs_Hotswap:Hotswap_MX_Plated_1.00u, F.Cu at (393.4, 173.9)
- added K_32: KEYSW, ScottoKeebs_Hotswap:Hotswap_MX_Plated_1.00u, F.Cu at (412.5, 173.9)
- added K_33: KEYSW, ScottoKeebs_Hotswap:Hotswap_MX_Plated_1.50u, F.Cu at (436.3, 173.9)
- added K_34: KEYSW, ScottoKeebs_Hotswap:Hotswap_MX_Plated_1.00u, F.Cu at (474.4, 173.9)
- added K_35: KEYSW, ScottoKeebs_Hotswap:Hotswap_MX_Plated_1.00u, F.Cu at (493.4, 173.9)
- added K_36: KEYSW, ScottoKeebs_Hotswap:Hotswap_MX_Plated_1.00u, F.Cu at (92.7, 192.9)
- added K_37: KEYSW, ScottoKeebs_Hotswap:Hotswap_MX_Plated_1.00u, F.Cu at (111.7, 192.9)
- added K_38: KEYSW, ScottoKeebs_Hotswap:Hotswap_MX_Plated_1.75u, F.Cu at (157.0, 192.9)
- added K_39: KEYSW, ScottoKeebs_Hotswap:Hotswap_MX_Plated_1.00u, F.Cu at (183.2, 192.9)
- added K_4: KEYSW, ScottoKeebs_Hotswap:Hotswap_MX_Plated_1.00u, F.Cu at (187.9, 154.8)
- added K_42: KEYSW, ScottoKeebs_Hotswap:Hotswap_MX_Plated_1.00u, F.Cu at (240.3, 192.9)
- added K_43: KEYSW, ScottoKeebs_Hotswap:Hotswap_MX_Plated_1.00u, F.Cu at (259.4, 192.9)
- added K_44: KEYSW, ScottoKeebs_Hotswap:Hotswap_MX_Plated_1.00u, F.Cu at (302.9, 192.9)
- added K_45: KEYSW, ScottoKeebs_Hotswap:Hotswap_MX_Plated_1.00u, F.Cu at (322.0, 192.9)
- added K_46: KEYSW, ScottoKeebs_Hotswap:Hotswap_MX_Plated_1.00u, F.Cu at (341.0, 192.9)
- added K_47: KEYSW, ScottoKeebs_Hotswap:Hotswap_MX_Plated_1.00u, F.Cu at (360.1, 192.9)
- added K_48: KEYSW, ScottoKeebs_Hotswap:Hotswap_MX_Plated_1.00u, F.Cu at (379.1, 192.9)
- added K_49: KEYSW, ScottoKeebs_Hotswap:Hotswap_MX_Plated_1.00u, F.Cu at (398.2, 192.9)
- added K_5: KEYSW, ScottoKeebs_Hotswap:Hotswap_MX_Plated_1.00u, F.Cu at (207.0, 154.8)
- added K_50: KEYSW, ScottoKeebs_Hotswap:Hotswap_MX_Plated_2.25u, F.Cu at (429.1, 192.9)
- added K_51: KEYSW, ScottoKeebs_Hotswap:Hotswap_MX_Plated_1.00u, F.Cu at (479.1, 192.9)
- added K_52: KEYSW, ScottoKeebs_Hotswap:Hotswap_MX_Plated_1.00u, F.Cu at (498.2, 192.9)
- added K_53: KEYSW, ScottoKeebs_Hotswap:Hotswap_MX_Plated_1.00u, F.Cu at (97.4, 212.0)
- added K_54: KEYSW, ScottoKeebs_Hotswap:Hotswap_MX_Plated_1.00u, F.Cu at (116.5, 212.0)
- added K_55: KEYSW, ScottoKeebs_Hotswap:Hotswap_MX_Plated_2.25u, F.Cu at (161.7, 212.0)
- added K_56: KEYSW, ScottoKeebs_Hotswap:Hotswap_MX_Plated_1.00u, F.Cu at (192.7, 212.0)
- added K_57: KEYSW, ScottoKeebs_Hotswap:Hotswap_MX_Plated_1.00u, F.Cu at (211.7, 212.0)
- added K_58: KEYSW, ScottoKeebs_Hotswap:Hotswap_MX_Plated_1.00u, F.Cu at (230.8, 212.0)
- added K_59: KEYSW, ScottoKeebs_Hotswap:Hotswap_MX_Plated_1.00u, F.Cu at (249.8, 212.0)
- added K_6: KEYSW, ScottoKeebs_Hotswap:Hotswap_MX_Plated_1.00u, F.Cu at (226.0, 154.8)
- added K_60: KEYSW, ScottoKeebs_Hotswap:Hotswap_MX_Plated_1.00u, F.Cu at (268.9, 212.0)
- added K_61: KEYSW, ScottoKeebs_Hotswap:Hotswap_MX_Plated_1.00u, F.Cu at (312.5, 212.0)
- added K_62: KEYSW, ScottoKeebs_Hotswap:Hotswap_MX_Plated_1.00u, F.Cu at (331.5, 212.0)
- added K_63: KEYSW, ScottoKeebs_Hotswap:Hotswap_MX_Plated_1.00u, F.Cu at (350.6, 212.0)
- added K_64: KEYSW, ScottoKeebs_Hotswap:Hotswap_MX_Plated_1.00u, F.Cu at (369.6, 212.0)
- added K_65: KEYSW, ScottoKeebs_Hotswap:Hotswap_MX_Plated_1.00u, F.Cu at (388.7, 212.0)
- added K_66: KEYSW, ScottoKeebs_Hotswap:Hotswap_MX_Plated_2.75u, F.Cu at (424.4, 212.0)
- added K_67: KEYSW, ScottoKeebs_Hotswap:Hotswap_MX_Plated_1.00u, F.Cu at (474.4, 212.0)
- added K_68: KEYSW, ScottoKeebs_Hotswap:Hotswap_MX_Plated_1.00u, F.Cu at (493.4, 212.0)
- added K_69: KEYSW, ScottoKeebs_Hotswap:Hotswap_MX_Plated_1.00u, F.Cu at (102.2, 231.0)
- added K_7: KEYSW, ScottoKeebs_Hotswap:Hotswap_MX_Plated_1.00u, F.Cu at (245.1, 154.8)
- added K_70: KEYSW, ScottoKeebs_Hotswap:Hotswap_MX_Plated_1.00u, F.Cu at (121.3, 231.0)
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Connections:
- K_40 pad 1: col5 -> col6
- K_41 pad 1: col6 -> col7
Other:
- board outline added: 430 x 143.2 mm

Commit message: Internalized wiring done.
Parts:
- moved D_17 6.58 mm to (497.1, 161.9)
- moved D_16 6.58 mm to (478.3, 161.9)
- moved U2 2.02 mm to (440.2, 114.3)
- moved U1 1.61 mm to (149.9, 114.5)
Connections:
- U1 pad 10: unconnected-(U1-9-Pad10) -> col4
- U1 pad 11: unconnected-(U1-10-Pad11) -> col3
- U1 pad 12: unconnected-(U1-11-Pad12) -> col2
- U1 pad 13: unconnected-(U1-12-Pad13) -> col1
- U1 pad 14: unconnected-(U1-13-Pad14) -> col0
- U1 pad 16: unconnected-(U1-15-Pad16) -> row0
- U1 pad 17: unconnected-(U1-26-Pad17) -> row1
- U1 pad 18: unconnected-(U1-27-Pad18) -> row2
- U1 pad 19: unconnected-(U1-28-Pad19) -> row3
- U1 pad 20: unconnected-(U1-29-Pad20) -> row4
- U1 pad 4: unconnected-(U1-3-Pad4) -> col10
- U1 pad 5: unconnected-(U1-4-Pad5) -> col9
- U1 pad 6: unconnected-(U1-5-Pad6) -> col8
- U1 pad 7: unconnected-(U1-6-Pad7) -> col7
- U1 pad 8: unconnected-(U1-7-Pad8) -> col6
- U1 pad 9: unconnected-(U1-8-Pad9) -> col5
- U2 pad 10: unconnected-(U2-9-Pad10) -> col21
- U2 pad 11: unconnected-(U2-10-Pad11) -> col20
- U2 pad 12: unconnected-(U2-11-Pad12) -> col18
- U2 pad 13: unconnected-(U2-12-Pad13) -> col17
- U2 pad 14: unconnected-(U2-13-Pad14) -> col16
- U2 pad 15: unconnected-(U2-14-Pad15) -> col15
- U2 pad 16: unconnected-(U2-15-Pad16) -> col14
- U2 pad 17: unconnected-(U2-26-Pad17) -> col13
- U2 pad 18: unconnected-(U2-27-Pad18) -> col12
- U2 pad 19: unconnected-(U2-28-Pad19) -> col11
- U2 pad 5: unconnected-(U2-4-Pad5) -> row9
- U2 pad 6: unconnected-(U2-5-Pad6) -> row8
- U2 pad 7: unconnected-(U2-6-Pad7) -> row7
- U2 pad 8: unconnected-(U2-7-Pad8) -> row6
- U2 pad 9: unconnected-(U2-8-Pad9) -> row5
Routing:
- net row4: track 0.00 -> 345.5 mm
- net row3: track 0.00 -> 336.9 mm
- net row8: track 0.00 -> 331.9 mm
- net row9: track 0.00 -> 323.1 mm
- net row7: track 0.00 -> 322.1 mm
- net row2: track 0.00 -> 308.9 mm
- net row1: track 0.00 -> 300.0 mm
- net row6: track 0.00 -> 284.0 mm
- net row5: track 0.00 -> 273.0 mm
- net row0: track 0.00 -> 269.6 mm
- net col11: track 0.00 -> 218.2 mm
- net col12: track 0.00 -> 216.9 mm
- net col8: track 0.00 -> 191.0 mm
- net col9: track 0.00 -> 188.1 mm
- net col14: track 0.00 -> 175.7 mm
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
Commit message: mounting holes placed
Parts:
- added ?: , , B.Cu at (478.7, 393.3)
- added REF**: MountingHole_2.2mm_M2, MountingHole:MountingHole_2.2mm_M2, F.Cu at (256.0, 231.7)
- added REF**: MountingHole_2.2mm_M2, MountingHole:MountingHole_2.2mm_M2, F.Cu at (187.9, 165.4)
- added REF**: Stabilizer_MX_2.00u, ScottoKeebs_Stabilizer:Stabilizer_MX_2.00u, F.Cu at (161.7, 212.0)
- added REF**: Stabilizer_Cherry_MX_3.00u, PCM_Mounting_Keyboard_Stabilizer:Stabilizer_Cherry_MX_3.00u, F.Cu at (322.0, 231.0)
- added REF**: Stabilizer_Cherry_MX_3.00u, PCM_Mounting_Keyboard_Stabilizer:Stabilizer_Cherry_MX_3.00u, F.Cu at (240.3, 231.0)
- added REF**: MountingHole_2.2mm_M2, MountingHole:MountingHole_2.2mm_M2, F.Cu at (263.7, 132.8)
- added REF**: MountingHole_2.2mm_M2, MountingHole:MountingHole_2.2mm_M2, B.Cu at (401.9, 207.0)
- added REF**: MountingHole_2.2mm_M2, MountingHole:MountingHole_2.2mm_M2, B.Cu at (381.8, 110.6)
- added REF**: MountingHole_2.2mm_M2, MountingHole:MountingHole_2.2mm_M2, B.Cu at (303.7, 134.4)
- added REF**: MountingHole_2.2mm_M2, MountingHole:MountingHole_2.2mm_M2, B.Cu at (308.7, 231.4)
- added REF**: MountingHole_2.2mm_M2, MountingHole:MountingHole_2.2mm_M2, B.Cu at (423.9, 167.2)
- added REF**: MountingHole_2.2mm_M2, MountingHole:MountingHole_2.2mm_M2, F.Cu at (266.3, 184.4)
- added REF**: MountingHole_2.2mm_M2, MountingHole:MountingHole_2.2mm_M2, B.Cu at (474.5, 135.2)
- added REF**: MountingHole_2.2mm_M2, MountingHole:MountingHole_2.2mm_M2, B.Cu at (506.1, 241.4)
- added REF**: MountingHole_2.2mm_M2, MountingHole:MountingHole_2.2mm_M2, B.Cu at (311.1, 183.2)
- added REF**: MountingHole_2.2mm_M2, MountingHole:MountingHole_2.2mm_M2, B.Cu at (478.7, 393.3)
- added REF**: Stabilizer_MX_2.00u, ScottoKeebs_Stabilizer:Stabilizer_MX_2.00u, F.Cu at (431.5, 154.8)
- added REF**: Stabilizer_MX_2.00u, ScottoKeebs_Stabilizer:Stabilizer_MX_2.00u, F.Cu at (429.1, 192.9)
- added REF**: MountingHole_2.2mm_M2, MountingHole:MountingHole_2.2mm_M2, F.Cu at (181.7, 208.4)
- added REF**: MountingHole_2.2mm_M2, MountingHole:MountingHole_2.2mm_M2, F.Cu at (86.7, 239.5)
- added REF**: Stabilizer_MX_2.00u, ScottoKeebs_Stabilizer:Stabilizer_MX_2.00u, F.Cu at (424.4, 212.0)
- added REF**: MountingHole_2.2mm_M2, MountingHole:MountingHole_2.2mm_M2, F.Cu at (208.3, 110.6)
- added REF**: MountingHole_2.2mm_M2, MountingHole:MountingHole_2.2mm_M2, F.Cu at (115.1, 132.3)
- K_15: footprint ScottoKeebs_Hotswap:Hotswap_MX_Plated_1.00u -> ScottoKeebs_Hotswap:Hotswap_MX_Plated_2.00u
Routing:
- net col18: track 113.7 -> 115.2 mm
