File: SplitSync/SplitSync.kicad_pcb (KiCad board)
At the start: 2 copper layers, 430 x 143.2 mm, 192 parts, among them U1 RP2040_Zero, U2 RP2040_Zero, U3 TRRS, U4 TRRS

Commit message: Logo added onto board
Parts:
- added G***: LOGO, CraftsByKris:Crafts_By_Kris, F.Cu at (396.5, 119.3)
- added G***: LOGO, CraftsByKris:Crafts_By_Kris, F.Cu at (194.9, 119.9)
- moved REF** 5.22 mm to (213.5, 110.1)
- moved REF** 4.81 mm to (377.0, 111.3)

Commit message: Flex Cuts
Parts:
- added REF**: RelieveCut, RelieveCut, F.Cu at (455.3, 173.3)
- added REF**: RelieveCut, RelieveCut, F.Cu at (455.4, 230.5)
- added REF**: RelieveCut, RelieveCut, F.Cu at (455.4, 192.4)
- added REF**: RelieveCut, RelieveCut, F.Cu at (237.8, 145.0)
- added REF**: RelieveCut, RelieveCut, F.Cu at (135.7, 210.5)
- added REF**: RelieveCut, RelieveCut, F.Cu at (135.7, 172.5)
- added REF**: RelieveCut, RelieveCut, F.Cu at (107.3, 145.3)
- added REF**: RelieveCut, RelieveCut, F.Cu at (479.1, 145.3)
- added REF**: RelieveCut, RelieveCut, F.Cu at (392.9, 137.9)
- added REF**: RelieveCut, RelieveCut, F.Cu at (135.7, 229.6)
- added REF**: RelieveCut, RelieveCut, F.Cu at (316.6, 138.0)
- added REF**: RelieveCut, RelieveCut, F.Cu at (455.3, 154.2)
- added REF**: RelieveCut, RelieveCut, F.Cu at (135.6, 191.4)
- added REF**: RelieveCut, RelieveCut, F.Cu at (256.9, 144.9)
- added REF**: RelieveCut, RelieveCut, F.Cu at (455.3, 211.3)
- added REF**: RelieveCut, RelieveCut, F.Cu at (218.9, 144.9)
- added REF**: RelieveCut, RelieveCut, F.Cu at (354.8, 137.9)
- added REF**: RelieveCut, RelieveCut, F.Cu at (335.7, 138.0)
- added REF**: RelieveCut, RelieveCut, F.Cu at (373.7, 138.0)
- added REF**: RelieveCut, RelieveCut, F.Cu at (199.7, 144.9)
- added REF**: RelieveCut, RelieveCut, F.Cu at (135.6, 153.3)

Commit message: final overview done
Parts:
- K_15: footprint ScottoKeebs_Hotswap:Hotswap_MX_Plated_2.00u -> ScottoKeebs_Hotswap:Hotswap_MX_Plated_1.00u
- moved REF** 0.54 mm to (354.8, 137.4)
- moved REF** 0.54 mm to (392.8, 137.4)
- moved REF** 0.54 mm to (316.6, 137.4)
- moved REF** 0.54 mm to (335.7, 137.4)
- moved REF** 0.54 mm to (373.7, 137.4)
- moved U3 0.10 mm to (263.1, 104.4)
Connections:
- U1 pad 1: unconnected-(U1-0-Pad1) -> Ring1
- U1 pad 2: unconnected-(U1-1-Pad2) -> Ring2
- U1 pad 22: unconnected-(U1-GND-Pad22) -> Sleeve
- U1 pad 23: unconnected-(U1-5V-Pad23) -> Tip
- U2 pad 1: unconnected-(U2-0-Pad1) -> Ring1_2
- U2 pad 2: unconnected-(U2-1-Pad2) -> Ring2_2
- U2 pad 22: unconnected-(U2-GND-Pad22) -> Sleeve_2
- U2 pad 23: unconnected-(U2-5V-Pad23) -> Tip_2
- U3 pad 1: unconnected-(U3-SLEEVE-Pad1) -> Sleeve
- U3 pad 2: unconnected-(U3-TIP-Pad2) -> Tip
- U3 pad 3: unconnected-(U3-RING1-Pad3) -> Ring1
- U3 pad 4: unconnected-(U3-RING2-Pad4) -> Ring2
- U4 pad 1: unconnected-(U4-SLEEVE-Pad1) -> Sleeve_2
- U4 pad 2: unconnected-(U4-TIP-Pad2) -> Tip_2
- U4 pad 3: unconnected-(U4-RING1-Pad3) -> Ring1_2
- U4 pad 4: unconnected-(U4-RING2-Pad4) -> Ring2_2
Routing:
- net Ring2_2: track 0.00 -> 162.7 mm
- net Ring1_2: track 0.00 -> 144.1 mm
- net Sleeve_2: track 0.00 -> 129.8 mm
- net Tip: track 0.00 -> 126.9 mm
- net Tip_2: track 0.00 -> 126.6 mm
- net Sleeve: track 0.00 -> 122.6 mm
- net Ring1: track 0.00 -> 119.9 mm
- net Ring2: track 0.00 -> 108.2 mm
