File: SplitSync/SplitSync.kicad_pcb (KiCad board)
At the start: 2 copper layers, 430 x 143.2 mm, 215 parts, among them U1 RP2040_Zero, U2 RP2040_Zero, U3 TRRS, U4 TRRS

Commit message: guide holes set for case building phase
Parts:
- removed ?: , 
- removed the REF** at (478.7, 393.3)
- added REF**: MountingHole_2.2mm_M2, MountingHole:MountingHole_2.2mm_M2, B.Cu at (467.1, 102.2)
- added REF**: MountingHole_2.2mm_M2, MountingHole:MountingHole_2.2mm_M2, B.Cu at (268.3, 244.7)
- added REF**: MountingHole_2.2mm_M2, MountingHole:MountingHole_2.2mm_M2, B.Cu at (80.6, 144.6)
- added REF**: MountingHole_2.2mm_M2, MountingHole:MountingHole_2.2mm_M2, B.Cu at (273.1, 102.7)
- added REF**: MountingHole_2.2mm_M2, MountingHole:MountingHole_2.2mm_M2, B.Cu at (510.3, 145.4)
- added REF**: MountingHole_2.2mm_M2, MountingHole:MountingHole_2.2mm_M2, B.Cu at (294.0, 244.7)
- added REF**: MountingHole_2.2mm_M2, MountingHole:MountingHole_2.2mm_M2, B.Cu at (123.0, 102.2)
- added REF**: MountingHole_2.2mm_M2, MountingHole:MountingHole_2.2mm_M2, B.Cu at (509.8, 244.7)
- added REF**: MountingHole_2.2mm_M2, MountingHole:MountingHole_2.2mm_M2, B.Cu at (81.0, 244.7)
- added REF**: MountingHole_2.2mm_M2, MountingHole:MountingHole_2.2mm_M2, B.Cu at (298.8, 102.7)
- moved REF** 0.34 mm to (505.8, 241.3)
