File: SplitSync/SplitSync.kicad_sch (KiCad schematic)
At the start: 168 parts, among them U1 RP2040_Zero, U2 RP2040_Zero, U3 TRRS, U4 TRRS

Commit message: final overview done
Connections:
- net Sleeve: now reaches U3.1 (SLEEVE)
- net Sleeve: now also U1.22 (GND)
- net Tip: now reaches U3.2 (TIP)
- net Tip: now also U1.23 (5V)
- net Ring1: now reaches U3.3 (RING1)
- net Ring1: now also U1.1 (0)
- net Ring2: now reaches U3.4 (RING2)
- net Ring2: now also U1.2 (1)
- net Ring1_2: now reaches U2.1 (0)
- net Ring1_2: now also U4.3 (RING1)
- net Ring2_2: now reaches U2.2 (1)
- net Ring2_2: now also U4.4 (RING2)
- net Sleeve_2: now reaches U2.22 (GND)
- net Sleeve_2: now also U4.1 (SLEEVE)
- net Tip_2: now reaches U2.23 (5V)
- net Tip_2: now also U4.2 (TIP)
- no-connect marks 0 -> 7
Other:
- moved on the sheet: U3, U4
